File: PCB/arcade/arcade.kicad_pcb (KiCad board)
At the start: 4 copper layers, 200.1 x 63 mm, 50 parts, among them J1 USB_C_Receptacle_USB2.0_16P, J10 USB3_A_Stacked, J11 USB_A_Stacked, J12 RJ45_RB1-125B8G1A, J13 HDMI_A_1.4, J15 Conn_02x24_Odd_Even, J16 Conn_02x24_Odd_Even, J2 Conn_02x03_Odd_Even, J3 Conn_02x06_Odd_Even, J4 Screw_Terminal_01x02, J5 Screw_Terminal_01x12, J6 Screw_Terminal_01x08, J7 Screw_Terminal_01x12, J8 Conn_01x02_Pin, J9 Conn_01x06_Pin, U1 RP2040, U10 TCA9548AMRGER, U2 TLC5947RHB, U3 TLC5947RHB, U4 TLC5947RHB, U5 ME6211C33M5, U6 CD74HC4067M, U7 CD74HC4067M, U8 W25Q16JVSS, U9 TS3USB221ARSERG4, Y3 Crystal_GND24

Commit message: board stuff
Parts:
- removed J10: USB3_A_Stacked, Connector_USB:USB3_A_Molex_48406-0001_Horizontal_Stacked
- removed J13: HDMI_A_1.4, Connector_Video:HDMI_A_Amphenol_10029449-x01xLF_Horizontal
- added C12: 100n, Capacitor_SMD:C_0402_1005Metric, F.Cu at (242.0, 152.8)
- added C13: 100n, Capacitor_SMD:C_0402_1005Metric, F.Cu at (242.0, 154.7)
- added C3: 100n, Capacitor_SMD:C_0402_1005Metric, F.Cu at (250.5, 91.4)
- added D2: LED Green, LED_SMD:LED_0603_1608Metric, F.Cu at (247.0, 91.7)
- added J17: Conn_01x03, Connector_PinHeader_2.54mm:PinHeader_1x03_P2.54mm_Vertical, F.Cu at (239.8, 81.3)
- added J18: THD-02-R, Connector_PinHeader_2.54mm:PinHeader_2x02_P2.54mm_Vertical, F.Cu at (244.4, 81.3)
- added J19: USB3_A, CM5IO:MTCONN_UBAF30-D2011, F.Cu at (162.0, 107.6)
- added J20: 690-019-298-412, CM5IO:EDAC 690-019-298-412, F.Cu at (180.9, 105.5)
- added J22: 690-019-298-412, CM5IO:EDAC 690-019-298-412, F.Cu at (200.9, 105.5)
- added R1: 1k, Resistor_SMD:R_0402_1005Metric, F.Cu at (243.5, 87.1)
- added R2: 470R, Resistor_SMD:R_0402_1005Metric, F.Cu at (243.5, 89.1)
- added R3: 470R, Resistor_SMD:R_0402_1005Metric, F.Cu at (243.5, 91.1)
- added R6: 2.2K 1%, Resistor_SMD:R_0402_1005Metric, F.Cu at (249.0, 148.1)
- added R7: 2.2K 1%, Resistor_SMD:R_0402_1005Metric, F.Cu at (249.0, 150.1)
- added TP3: TestPoint, TestPoint:TestPoint_Pad_2.0x2.0mm, F.Cu at (239.5, 90.7)
- added U11: RP2350A, Package_DFN_QFN:QFN-60-1EP_7x7mm_P0.4mm_EP3.4x3.4mm, F.Cu at (41.9, 105.8)
- added U12: MagJack-A70-112-331N126, CM5IO:TRJG0926HENL, F.Cu at (142.5, 106.0)
- added U13: RT9742SNGV, Package_TO_SOT_SMD:TSOT-23_HandSoldering, F.Cu at (244.1, 149.6)
- added U9: TS3USB221ARSERG4, TS3USB221A:RSE10, F.Cu at (62.5, 101.5)
- J11: value USB_A_Stacked -> USB_C_Receptacle_USB2.0_16P; footprint Connector_USB:USB_A_CUI_UJ2-ADH-TH_Horizontal_Stacked -> Connector_USB:USB_C_Receptacle_GCT_USB4110
- J12: value RJ45_RB1-125B8G1A -> THD-02-R; footprint Connector_RJ:RJ45_UDE_RB1-125B8G1A -> Connector_PinHeader_2.54mm:PinHeader_2x02_P2.54mm_Vertical
- U1: value RP2040 -> TPD4EUSB30; footprint Package_DFN_QFN:QFN-56-1EP_7x7mm_P0.4mm_EP3.2x3.2mm -> Package_SON:USON-10_2.5x1.0mm_P0.5mm
- U10: value TCA9548AMRGER -> TPD4EUSB30; footprint Package_DFN_QFN:Texas_RGE0024C_VQFN-24-1EP_4x4mm_P0.5mm_EP2.1x2.1mm -> Package_SON:USON-10_2.5x1.0mm_P0.5mm
- moved U1 205.3 mm to (246.5, 88.4)
- moved U10 168.4 mm to (249.4, 88.4)
- moved J12 112.4 mm to (235.7, 149.4)
- moved J11 31.4 mm to (137.5, 80.5)
- moved J2 22.0 mm to (160.0, 65.5)
- moved J4 13.0 mm to (182.0, 57.3)
- moved Module1 2.92 mm to (218.5, 63.0)
- moved C18 0.20 mm to (43.8, 112.5)
- moved R10 0.20 mm to (42.1, 112.5)
Connections:
- C1 pad 2: /GND -> GND
- C15 pad 2: /GND -> GND
- C16 pad 2: /GND -> GND
- C17 pad 1: /GND -> GND
- C18 pad 1: /GND -> GND
- C19 pad 1: /GND -> GND
- C2 pad 2: /GND -> GND
- C20 pad 1: /GND -> GND
- C21 pad 1: /GND -> GND
- C22 pad 1: /GND -> GND
- C23 pad 1: /GND -> GND
- C24 pad 2: /GND -> GND
- C6 pad 2: /GND -> GND
- D1 pad 3: /GND -> GND
- J1 pad A1: /GND -> GND
- J1 pad A12: /GND -> GND
- J1 pad B1: /GND -> GND
- J1 pad B12: /GND -> GND
- J1 pad S1: /GND -> GND
- J11 pad SH: unconnected-(J11-Shield-PadSH) -> (no net)
- J2 pad 1: /GND -> GND
- J2 pad 2: /GND -> GND
- J3 pad 11: /GND -> GND
- J3 pad 12: /GND -> GND
- J4 pad 1: /GND -> GND
- J9 pad 6: /GND -> GND
- Module1 pad 1: unconnected-(Module1A-GND-Pad1) -> GND
- Module1 pad 10: unconnected-(Module1A-Ethernet_Pair0_N-Pad10) -> /TRD0_N
- Module1 pad 100: unconnected-(Module1A-CAM_GPIO1-Pad100) -> /CAM_GPIO1
- Module1 pad 101: unconnected-(Module1B-USB_OTG_ID-Pad101) -> /USBOTG_ID
- Module1 pad 102: unconnected-(Module1B-PCIe_nCLKREQ-Pad102) -> /PCIE_nCLKREQ
- Module1 pad 103: unconnected-(Module1B-USB2_N-Pad103) -> /USB2_N
- Module1 pad 104: unconnected-(Module1B-PCIE_nWAKE-Pad104) -> /PCIE_nWAKE
- Module1 pad 105: unconnected-(Module1B-USB2_P-Pad105) -> /USB2_P
- Module1 pad 106: unconnected-(Module1B-PCIE_PWR_EN-Pad106) -> /PCIE_PWR_EN
- Module1 pad 107: unconnected-(Module1B-GND-Pad107) -> GND
- Module1 pad 108: unconnected-(Module1B-GND-Pad108) -> GND
- Module1 pad 109: unconnected-(Module1B-PCIe_nRST-Pad109) -> /PCIE_nRST
- Module1 pad 11: unconnected-(Module1A-Ethernet_Pair2_P-Pad11) -> /TRD2_P
- Module1 pad 110: unconnected-(Module1B-PCIe_CLK_P-Pad110) -> /PCIE_CLK_P
- Module1 pad 111: unconnected-(Module1B-VBUS_EN-Pad111) -> /VBUS_EN
- Module1 pad 112: unconnected-(Module1B-PCIe_CLK_N-Pad112) -> /PCIE_CLK_N
- Module1 pad 113: unconnected-(Module1B-GND-Pad113) -> GND
- Module1 pad 114: unconnected-(Module1B-GND-Pad114) -> GND
- Module1 pad 115: unconnected-(Module1B-MIPI0_D0_N-Pad115) -> /DPHY0_D0_N
- Module1 pad 116: unconnected-(Module1B-PCIe_RX_P-Pad116) -> /PCIE_RX_P
- Module1 pad 117: unconnected-(Module1B-MIPI0_D0_P-Pad117) -> /DPHY0_D0_P
- Module1 pad 118: unconnected-(Module1B-PCIe_RX_N-Pad118) -> /PCIE_RX_N
- Module1 pad 119: unconnected-(Module1B-GND-Pad119) -> GND
- Module1 pad 12: unconnected-(Module1A-Ethernet_Pair0_P-Pad12) -> /TRD0_P
- Module1 pad 120: unconnected-(Module1B-GND-Pad120) -> GND
- Module1 pad 121: unconnected-(Module1B-MIPI0_D1_N-Pad121) -> /DPHY0_D1_N
- Module1 pad 122: unconnected-(Module1B-PCIe_TX_P-Pad122) -> /PCIE_TX_P
- Module1 pad 123: unconnected-(Module1B-MIPI0_D1_P-Pad123) -> /DPHY0_D1_P
- Module1 pad 124: unconnected-(Module1B-PCIe_TX_N-Pad124) -> /PCIE_TX_N
- Module1 pad 125: unconnected-(Module1B-GND-Pad125) -> GND
- Module1 pad 126: unconnected-(Module1B-GND-Pad126) -> GND
- Module1 pad 127: unconnected-(Module1B-MIPI0_C_N-Pad127) -> /DPHY0_C_N
- Module1 pad 128: unconnected-(Module1B-USB3-0-RX_N-Pad128) -> /USB3-0-RX_N
- Module1 pad 129: unconnected-(Module1B-MIPI0_C_P-Pad129) -> /DPHY0_C_P
- Module1 pad 13: unconnected-(Module1A-GND-Pad13) -> GND
- Module1 pad 130: unconnected-(Module1B-USB3-0-RX_P-Pad130) -> /USB3-0-RX_P
- Module1 pad 131: unconnected-(Module1B-GND-Pad131) -> GND
- Module1 pad 132: unconnected-(Module1B-GND-Pad132) -> GND
- Module1 pad 133: unconnected-(Module1B-MIPI0_D2_N-Pad133) -> /DPHY0_D2_N
- Module1 pad 134: unconnected-(Module1B-USB3-0-D_P-Pad134) -> /USB3-0-D_P
- Module1 pad 135: unconnected-(Module1B-MIPI0_D2_P-Pad135) -> /DPHY0_D2_P
- Module1 pad 136: unconnected-(Module1B-USB3-0-D_N-Pad136) -> /USB3-0-D_N
- Module1 pad 137: unconnected-(Module1B-GND-Pad137) -> GND
- Module1 pad 138: unconnected-(Module1B-GND-Pad138) -> GND
- Module1 pad 139: unconnected-(Module1B-MIPI0_D3_N-Pad139) -> /DPHY0_D3_N
- Module1 pad 14: unconnected-(Module1A-GND-Pad14) -> GND
- Module1 pad 140: unconnected-(Module1B-USB3-0-TX_N-Pad140) -> /USB3-0-TX_N
- Module1 pad 141: unconnected-(Module1B-MIPI0_D3_P-Pad141) -> /DPHY0_D3_P
- Module1 pad 142: unconnected-(Module1B-USB3-0-TX_P-Pad142) -> /USB3-0-TX_P
- Module1 pad 143: unconnected-(Module1B-HDMI1_HOTPLUG-Pad143) -> /HDMI1_HOTPLUG
- Module1 pad 144: unconnected-(Module1B-GND-Pad144) -> GND
- Module1 pad 145: unconnected-(Module1B-HDMI1_SDA-Pad145) -> /HDMI1_SDA
- Module1 pad 146: unconnected-(Module1B-HDMI1_TX2_P-Pad146) -> /HDMI1_D2_P
- Module1 pad 147: unconnected-(Module1B-HDMI1_SCL-Pad147) -> /HDMI1_SCL
- Module1 pad 148: unconnected-(Module1B-HDMI1_TX2_N-Pad148) -> /HDMI1_D2_N
- Module1 pad 149: unconnected-(Module1B-HDMI1_CEC-Pad149) -> /HDMI1_CEC
- Module1 pad 15: unconnected-(Module1A-Ethernet_nLED3(3.3v)-Pad15) -> /ETH_LEDY
- Module1 pad 150: unconnected-(Module1B-GND-Pad150) -> GND
- Module1 pad 151: unconnected-(Module1B-HDMI0_CEC-Pad151) -> /HDMI0_CEC
- Module1 pad 152: unconnected-(Module1B-HDMI1_TX1_P-Pad152) -> /HDMI1_D1_P
- Module1 pad 153: unconnected-(Module1B-HDMI0_HOTPLUG-Pad153) -> /HDMI0_HOTPLUG
- Module1 pad 154: unconnected-(Module1B-HDMI1_TX1_N-Pad154) -> /HDMI1_D1_N
- Module1 pad 155: unconnected-(Module1B-GND-Pad155) -> GND
- Module1 pad 156: unconnected-(Module1B-GND-Pad156) -> GND
- Module1 pad 157: unconnected-(Module1B-USB3-1-RX_N-Pad157) -> /USB3-1-RX_N
- Module1 pad 158: unconnected-(Module1B-HDMI1_TX0_P-Pad158) -> /HDMI1_D0_P
- Module1 pad 159: unconnected-(Module1B-USB3-1-RX_P-Pad159) -> /USB3-1-RX_P
- Module1 pad 16: unconnected-(Module1A-FAN_TACHO-Pad16) -> /TACHO
- Module1 pad 160: unconnected-(Module1B-HDMI1_TX0_N-Pad160) -> /HDMI1_D0_N
- Module1 pad 161: unconnected-(Module1B-GND-Pad161) -> GND
- Module1 pad 162: unconnected-(Module1B-GND-Pad162) -> GND
- Module1 pad 163: unconnected-(Module1B-USB3-1-D_P-Pad163) -> /USB3-1-D_P
- Module1 pad 164: unconnected-(Module1B-HDMI1_CLK_P-Pad164) -> /HDMI1_CK_P
- Module1 pad 165: unconnected-(Module1B-USB3-1-D_N-Pad165) -> /USB3-1-D_N
- Module1 pad 166: unconnected-(Module1B-HDMI1_CLK_N-Pad166) -> /HDMI1_CK_N
- Module1 pad 167: unconnected-(Module1B-GND-Pad167) -> GND
- Module1 pad 168: unconnected-(Module1B-GND-Pad168) -> GND
- Module1 pad 169: unconnected-(Module1B-USB3-1-TX_N-Pad169) -> /USB3-1-TX_N
- Module1 pad 17: unconnected-(Module1A-Ethernet_nLED2(3.3v)-Pad17) -> /ETH_LEDG
- Module1 pad 170: unconnected-(Module1B-HDMI0_TX2_P-Pad170) -> /HDMI0_D2_P
- Module1 pad 171: unconnected-(Module1B-USB3-1-TX_P-Pad171) -> /USB3-1-TX_P
- Module1 pad 172: unconnected-(Module1B-HDMI0_TX2_N-Pad172) -> /HDMI0_D2_N
- Module1 pad 173: unconnected-(Module1B-GND-Pad173) -> GND
- Module1 pad 174: unconnected-(Module1B-GND-Pad174) -> GND
- Module1 pad 175: unconnected-(Module1B-MIPI1_D0_N-Pad175) -> /DPHY1_D0_N
- Module1 pad 176: unconnected-(Module1B-HDMI0_TX1_P-Pad176) -> /HDMI0_D1_P
- Module1 pad 177: unconnected-(Module1B-MIPI1_D0_P-Pad177) -> /DPHY1_D0_P
- Module1 pad 178: unconnected-(Module1B-HDMI0_TX1_N-Pad178) -> /HDMI0_D1_N
- Module1 pad 179: unconnected-(Module1B-GND-Pad179) -> GND
- Module1 pad 18: unconnected-(Module1A-Ethernet_SYNC_OUT(3.3v)-Pad18) -> /SYNC_OUT
- Module1 pad 180: unconnected-(Module1B-GND-Pad180) -> GND
- Module1 pad 181: unconnected-(Module1B-MIPI1_D1_N-Pad181) -> /DPHY1_D1_N
- Module1 pad 182: unconnected-(Module1B-HDMI0_TX0_P-Pad182) -> /HDMI0_D0_P
- Module1 pad 183: unconnected-(Module1B-MIPI1_D1_P-Pad183) -> /DPHY1_D1_P
- Module1 pad 184: unconnected-(Module1B-HDMI0_TX0_N-Pad184) -> /HDMI0_D0_N
- Module1 pad 185: unconnected-(Module1B-GND-Pad185) -> GND
- Module1 pad 186: unconnected-(Module1B-GND-Pad186) -> GND
- Module1 pad 187: unconnected-(Module1B-MIPI1_C_N-Pad187) -> /DPHY1_C_N
- Module1 pad 188: unconnected-(Module1B-HDMI0_CLK_P-Pad188) -> /HDMI0_CK_P
- Module1 pad 189: unconnected-(Module1B-MIPI1_C_P-Pad189) -> /DPHY1_C_P
- Module1 pad 19: unconnected-(Module1A-FAN_PWM-Pad19) -> /PWM
- Module1 pad 190: unconnected-(Module1B-HDMI0_CLK_N-Pad190) -> /HDMI0_CK_N
- Module1 pad 191: unconnected-(Module1B-GND-Pad191) -> GND
- Module1 pad 192: unconnected-(Module1B-GND-Pad192) -> GND
- Module1 pad 193: unconnected-(Module1B-MIPI1_D2_N-Pad193) -> /DPHY1_D2_N
- Module1 pad 194: unconnected-(Module1B-MIPI1_D3_N-Pad194) -> /DPHY1_D3_N
- Module1 pad 195: unconnected-(Module1B-MIPI1_D2_P-Pad195) -> /DPHY1_D2_P
- Module1 pad 196: unconnected-(Module1B-MIPI1_D3_P-Pad196) -> /DPHY1_D3_P
- Module1 pad 197: unconnected-(Module1B-GND-Pad197) -> GND
- Module1 pad 198: unconnected-(Module1B-GND-Pad198) -> GND
- Module1 pad 199: unconnected-(Module1B-HDMI0_SDA-Pad199) -> /HDMI0_SDA
- Module1 pad 2: unconnected-(Module1A-GND-Pad2) -> GND
- Module1 pad 20: unconnected-(Module1A-EEPROM_nWP-Pad20) -> /EEPROM_nWP
- Module1 pad 200: unconnected-(Module1B-HDMI0_SCL-Pad200) -> /HDMI0_SCL
- Module1 pad 21: unconnected-(Module1A-LED_nACT-Pad21) -> Net-(Module1A-LED_nACT)
- Module1 pad 22: unconnected-(Module1A-GND-Pad22) -> GND
- Module1 pad 23: unconnected-(Module1A-GND-Pad23) -> GND
- Module1 pad 24: unconnected-(Module1A-GPIO26-Pad24) -> /GPIO26
- Module1 pad 25: unconnected-(Module1A-GPIO21-Pad25) -> /GPIO21
- Module1 pad 26: unconnected-(Module1A-GPIO19-Pad26) -> /GPIO19
- Module1 pad 27: unconnected-(Module1A-GPIO20-Pad27) -> /GPIO20
- Module1 pad 28: unconnected-(Module1A-GPIO13-Pad28) -> /GPIO13
- Module1 pad 29: unconnected-(Module1A-GPIO16-Pad29) -> /GPIO16
- Module1 pad 3: unconnected-(Module1A-Ethernet_Pair3_P-Pad3) -> /TRD3_P
- Module1 pad 30: unconnected-(Module1A-GPIO6-Pad30) -> /GPIO6
- Module1 pad 31: unconnected-(Module1A-GPIO12-Pad31) -> /GPIO12
- Module1 pad 32: unconnected-(Module1A-GND-Pad32) -> GND
- Module1 pad 33: unconnected-(Module1A-GND-Pad33) -> GND
- Module1 pad 34: unconnected-(Module1A-GPIO5-Pad34) -> /GPIO5
- Module1 pad 35: unconnected-(Module1A-ID_SC-Pad35) -> /ID_SC
- Module1 pad 36: unconnected-(Module1A-ID_SD-Pad36) -> /ID_SD
- Module1 pad 37: unconnected-(Module1A-GPIO7-Pad37) -> /GPIO7
- Module1 pad 38: unconnected-(Module1A-GPIO11-Pad38) -> /GPIO11
- Module1 pad 39: unconnected-(Module1A-GPIO8-Pad39) -> /GPIO8
- Module1 pad 4: unconnected-(Module1A-Ethernet_Pair1_P-Pad4) -> /TRD1_P
- Module1 pad 40: unconnected-(Module1A-GPIO9-Pad40) -> /GPIO9
- Module1 pad 41: unconnected-(Module1A-GPIO25-Pad41) -> /GPIO25
- Module1 pad 42: unconnected-(Module1A-GND-Pad42) -> GND
- Module1 pad 43: unconnected-(Module1A-GND-Pad43) -> GND
- Module1 pad 44: unconnected-(Module1A-GPIO10-Pad44) -> /GPIO10
- Module1 pad 45: unconnected-(Module1A-GPIO24-Pad45) -> /GPIO24
- Module1 pad 46: unconnected-(Module1A-GPIO22-Pad46) -> /GPIO22
- Module1 pad 47: unconnected-(Module1A-GPIO23-Pad47) -> /GPIO23
- Module1 pad 48: unconnected-(Module1A-GPIO27-Pad48) -> /GPIO27
- Module1 pad 49: unconnected-(Module1A-GPIO18-Pad49) -> /GPIO18
- Module1 pad 5: unconnected-(Module1A-Ethernet_Pair3_N-Pad5) -> /TRD3_N
- Module1 pad 50: unconnected-(Module1A-GPIO17-Pad50) -> /GPIO17
- Module1 pad 51: unconnected-(Module1A-GPIO15-Pad51) -> /GPIO15
- Module1 pad 52: unconnected-(Module1A-GND-Pad52) -> GND
- Module1 pad 53: unconnected-(Module1A-GND-Pad53) -> GND
- Module1 pad 54: unconnected-(Module1A-GPIO4-Pad54) -> /GPIO4
- Module1 pad 55: unconnected-(Module1A-GPIO14-Pad55) -> /GPIO14
- Module1 pad 56: unconnected-(Module1A-GPIO3-Pad56) -> /GPIO3
- Module1 pad 57: unconnected-(Module1A-SD_CLK-Pad57) -> /SD_CLK
- Module1 pad 58: unconnected-(Module1A-GPIO2-Pad58) -> /GPIO2
- Module1 pad 59: unconnected-(Module1A-GND-Pad59) -> GND
- Module1 pad 6: unconnected-(Module1A-Ethernet_Pair1_N-Pad6) -> /TRD1_N
- Module1 pad 60: unconnected-(Module1A-GND-Pad60) -> GND
- Module1 pad 61: unconnected-(Module1A-SD_DAT3-Pad61) -> /SD_DAT3
- Module1 pad 62: unconnected-(Module1A-SD_CMD-Pad62) -> /SD_CMD
- Module1 pad 63: unconnected-(Module1A-SD_DAT0-Pad63) -> /SD_DAT0
- Module1 pad 65: unconnected-(Module1A-GND-Pad65) -> GND
- Module1 pad 66: unconnected-(Module1A-GND-Pad66) -> GND
- Module1 pad 67: unconnected-(Module1A-SD_DAT1-Pad67) -> /SD_DAT1
- Module1 pad 69: unconnected-(Module1A-SD_DAT2-Pad69) -> /SD_DAT2
- Module1 pad 7: unconnected-(Module1A-GND-Pad7) -> GND
- Module1 pad 71: unconnected-(Module1A-GND-Pad71) -> GND
- Module1 pad 74: unconnected-(Module1A-GND-Pad74) -> GND
- Module1 pad 75: unconnected-(Module1A-SD_PWR_ON-Pad75) -> /SD_PWR_ON
- Module1 pad 76: unconnected-(Module1A-VBAT-Pad76) -> /VBAT
- Module1 pad 77: unconnected-(Module1A-+5v_(Input)-Pad77) -> /+5v
- Module1 pad 78: unconnected-(Module1A-GPIO_VREF(1.8v/3.3v_Input)-Pad78) -> /GPIO_VREF
- Module1 pad 79: unconnected-(Module1A-+5v_(Input)-Pad79) -> /+5v
- Module1 pad 8: unconnected-(Module1A-GND-Pad8) -> GND
- Module1 pad 80: unconnected-(Module1A-SCL0-Pad80) -> /SCL0
- Module1 pad 81: unconnected-(Module1A-+5v_(Input)-Pad81) -> /+5v
- Module1 pad 82: unconnected-(Module1A-SDA0-Pad82) -> /SDA0
- Module1 pad 83: unconnected-(Module1A-+5v_(Input)-Pad83) -> /+5v
- Module1 pad 84: unconnected-(Module1A-+3.3v_(Output)-Pad84) -> /+3.3v
- Module1 pad 85: unconnected-(Module1A-+5v_(Input)-Pad85) -> /+5v
- Module1 pad 86: unconnected-(Module1A-+3.3v_(Output)-Pad86) -> /+3.3v
- Module1 pad 87: unconnected-(Module1A-+5v_(Input)-Pad87) -> /+5v
- Module1 pad 88: unconnected-(Module1A-+1.8v_(Output)-Pad88) -> /+1.8v
- Module1 pad 89: unconnected-(Module1A-WiFi_nDisable-Pad89) -> /WL_nDis
- Module1 pad 9: unconnected-(Module1A-Ethernet_Pair2_N-Pad9) -> /TRD2_N
- Module1 pad 90: unconnected-(Module1A-+1.8v_(Output)-Pad90) -> /+1.8v
- Module1 pad 91: unconnected-(Module1A-BT_nDisable-Pad91) -> /BT_nDis
- Module1 pad 92: unconnected-(Module1A-PWR_BUT-Pad92) -> /PWR_BUT
- Module1 pad 93: unconnected-(Module1A-nRPIBOOT-Pad93) -> /nRPIBOOT
- Module1 pad 94: unconnected-(Module1A-CC1-Pad94) -> /CC1
- Module1 pad 95: unconnected-(Module1A-LED_nPWR-Pad95) -> /nPWR_LED
- Module1 pad 96: unconnected-(Module1A-CC2-Pad96) -> /CC2
- Module1 pad 97: unconnected-(Module1A-CAM_GPIO0-Pad97) -> /CAM_GPIO0
- Module1 pad 98: unconnected-(Module1A-GND-Pad98) -> GND
- Module1 pad 99: unconnected-(Module1A-PMIC_ENABLE-Pad99) -> /PMIC_ENABLE
- R11 pad 1: Net-(U1-USB_DM) -> Net-(U11-USB_DM)
- R12 pad 1: Net-(U1-USB_DP) -> Net-(U11-USB_DP)
- R4 pad 2: /GND -> GND
- R5 pad 2: /GND -> GND
- U1 pad 1: /3.3v -> /TRD3_P
- U1 pad 10: /3.3v -> /TRD3_P
- U1 pad 2: unconnected-(U1-GPIO0-Pad2) -> /TRD3_N
- U1 pad 3: unconnected-(U1-GPIO1-Pad3) -> GND
- U1 pad 4: unconnected-(U1-GPIO2-Pad4) -> /TRD2_N
- U1 pad 5: unconnected-(U1-GPIO3-Pad5) -> /TRD2_P
- U1 pad 6: unconnected-(U1-GPIO4-Pad6) -> /TRD2_P
- U1 pad 7: unconnected-(U1-GPIO5-Pad7) -> /TRD2_N
- U1 pad 8: unconnected-(U1-GPIO6-Pad8) -> GND
- U1 pad 9: unconnected-(U1-GPIO7-Pad9) -> /TRD3_N
- U10 pad 1: unconnected-(U10-SD0-Pad1) -> /TRD1_P
- U10 pad 10: unconnected-(U10-SD4-Pad10) -> /TRD1_P
- U10 pad 2: unconnected-(U10-SC0-Pad2) -> /TRD1_N
- U10 pad 3: unconnected-(U10-SD1-Pad3) -> GND
- U10 pad 4: unconnected-(U10-SC1-Pad4) -> /TRD0_N
- U10 pad 5: unconnected-(U10-SD2-Pad5) -> /TRD0_P
- U10 pad 6: unconnected-(U10-SC2-Pad6) -> /TRD0_P
- U10 pad 7: unconnected-(U10-SD3-Pad7) -> /TRD0_N
- U10 pad 8: unconnected-(U10-SC3-Pad8) -> GND
- U10 pad 9: unconnected-(U10-GND-Pad9) -> /TRD1_N
- U2 pad 29: /GND -> GND
- U2 pad 33: /GND -> GND
- U3 pad 29: /GND -> GND
- U3 pad 33: /GND -> GND
- U4 pad 29: /GND -> GND
- U4 pad 33: /GND -> GND
- U5 pad 2: /GND -> GND
- U6 pad 12: /GND -> GND
- U7 pad 12: /GND -> GND
- U8 pad 4: /GND -> GND
- Y3 pad 2: /GND -> GND
- Y3 pad 4: /GND -> GND
Routing:
- net /VBUS: track 66.0 -> 13.7 mm, vias 13 -> 14
- net GND: track 0.00 -> 50.5 mm, vias 0 -> 31
- net /GND: track 47.6 -> 0.00 mm, vias 31 -> 0
- net /EXT_5V: track 343.3 -> 371.7 mm
- net /3.3v: track 138.6 -> 120.0 mm, vias 3 -> 9
- net Net-(U11-DVDD-Pad23): track 0.00 -> 15.4 mm
- net Net-(U1-DVDD-Pad23): track 10.6 -> 0.00 mm
- net Net-(J1-CC1): track 0.00 -> 4.12 mm
- net Net-(C23-Pad2): track 7.54 -> 4.21 mm
- net Net-(J16-Pin_37): track 22.1 -> 19.5 mm
- net Net-(J16-Pin_41): track 25.1 -> 22.6 mm
- net Net-(U11-USB_DM): track 0.00 -> 2.43 mm
- net Net-(J16-Pin_43): track 27.8 -> 25.4 mm
- net Net-(J16-Pin_45): track 30.4 -> 28.1 mm
- net Net-(U1-USB_DM): track 1.92 -> 0.00 mm
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- added copper zone on In1.Cu, net /3.3v
- added copper zone on In1.Cu, net /VBUS
- added copper zone on In2.Cu, net GND
- removed copper zone on In2.Cu, net /GND
Other:
- outline, holes or cut-outs redrawn
