File: PCB/arcade/arcade.kicad_sch (KiCad schematic)
At the start: 49 parts, among them J1 USB_C_Receptacle_USB2.0_16P, J10 USB3_A_Stacked, J11 USB_A_Stacked, J13 HDMI_A_1.4, J15 Conn_02x24_Odd_Even, J16 Conn_02x24_Odd_Even, J2 Conn_02x03_Odd_Even, J3 Conn_02x06_Odd_Even, J4 Screw_Terminal_01x02, J5 Screw_Terminal_01x12, J6 Screw_Terminal_01x08, J7 Screw_Terminal_01x12, J8 Conn_01x02_Pin, J9 Conn_01x06_Pin, U1 RP2040, U10 TCA9548AMRGER, U2 TLC5947RHB, U3 TLC5947RHB, U4 TLC5947RHB, U5 ME6211C33M5, U6 CD74HC4067M, U7 CD74HC4067M, U8 W25Q16JVSS, U9 TS3USB221ARSERG4, Y3 Crystal_GND24

Commit message: board stuff
Parts:
- removed J10: USB3_A_Stacked, Connector_USB:USB3_A_Molex_48406-0001_Horizontal_Stacked, symbol Connector:USB3_A_Stacked
- removed J11: USB_A_Stacked, Connector_USB:USB_A_CUI_UJ2-ADH-TH_Horizontal_Stacked, symbol Connector:USB_A_Stacked
- removed J13: HDMI_A_1.4, Connector_Video:HDMI_A_Amphenol_10029449-x01xLF_Horizontal, symbol Connector:HDMI_A_1.4
- removed U1: RP2040, Package_DFN_QFN:QFN-56-1EP_7x7mm_P0.4mm_EP3.2x3.2mm, symbol MCU_RaspberryPi:RP2040
- removed U10: TCA9548AMRGER, Package_DFN_QFN:Texas_RGE0024C_VQFN-24-1EP_4x4mm_P0.5mm_EP2.1x2.1mm, symbol Interface_Expansion:TCA9548AMRGER
- added C12, C13, C3: 100n, Capacitor_SMD:C_0402_1005Metric, symbol Device:C
- added D2: LED Green, LED_SMD:LED_0603_1608Metric, symbol Device:LED
- added J11: USB_C_Receptacle_USB2.0_16P, Connector_USB:USB_C_Receptacle_GCT_USB4110, symbol Connector:USB_C_Receptacle_USB2.0_16P
- added J12, J18: THD-02-R, Connector_PinHeader_2.54mm:PinHeader_2x02_P2.54mm_Vertical, symbol Connector_Generic:Conn_02x02_Odd_Even
- added J17: Conn_01x03, Connector_PinHeader_2.54mm:PinHeader_1x03_P2.54mm_Vertical, symbol Connector_Generic:Conn_01x03
- added J19: USB3_A, CM5IO:MTCONN_UBAF30-D2011, symbol CM5IO:USB3_A
- added J20, J22: 690-019-298-412, CM5IO:EDAC 690-019-298-412, symbol CM5IO:HDMI_A_1.4
- added R1: 1k, Resistor_SMD:R_0402_1005Metric, symbol Device:R
- added R2, R3: 470R, Resistor_SMD:R_0402_1005Metric, symbol Device:R
- added R6, R7: 2.2K 1%, Resistor_SMD:R_0402_1005Metric, symbol Device:R
- added TP3: TestPoint, TestPoint:TestPoint_Pad_2.0x2.0mm, symbol Connector:TestPoint
- added U1, U10: TPD4EUSB30, Package_SON:USON-10_2.5x1.0mm_P0.5mm, symbol CM5IO:TPD4EUSB30
- added U11: RP2350A, Package_DFN_QFN:QFN-60-1EP_7x7mm_P0.4mm_EP3.4x3.4mm, symbol MCU_RaspberryPi:RP2350A
- added U12: MagJack-A70-112-331N126, CM5IO:TRJG0926HENL, symbol CM5IO:MagJack-A70-112-331N126
- added U13: RT9742SNGV, Package_TO_SOT_SMD:TSOT-23_HandSoldering, symbol CM5IO:RT9742SNGV
Connections:
- net 3.3v: now also U11.1 (IOVDD), U11.11 (IOVDD), U11.20 (IOVDD), U11.30 (IOVDD), U11.38 (IOVDD), U11.45 (IOVDD)
- net GND: now also Module1.1 (GND), Module1.107 (GND), Module1.108 (GND), Module1.113 (GND), Module1.114 (GND), Module1.119 (GND), Module1.120 (GND), Module1.125 (GND), Module1.126 (GND), Module1.13 (GND), Module1.131 (GND), Module1.132 (GND), Module1.137 (GND), Module1.138 (GND), Module1.14 (GND), Module1.144 (GND), Module1.150 (GND), Module1.155 (GND), Module1.156 (GND), Module1.161 (GND), Module1.162 (GND), Module1.167 (GND), Module1.168 (GND), Module1.173 (GND), Module1.174 (GND), Module1.179 (GND), Module1.180 (GND), Module1.185 (GND), Module1.186 (GND), Module1.191 (GND), Module1.192 (GND), Module1.197 (GND), Module1.198 (GND), Module1.2 (GND), Module1.22 (GND), Module1.23 (GND), Module1.32 (GND), Module1.33 (GND), Module1.42 (GND), Module1.43 (GND), Module1.52 (GND), Module1.53 (GND), Module1.59 (GND), Module1.60 (GND), Module1.65 (GND), Module1.66 (GND), Module1.7 (GND), Module1.71 (GND), Module1.74 (GND), Module1.8 (GND), Module1.98 (GND), C12.2, C13.2, C3.2, J17.2 (Pin_2), J19.10 (SHIELD), J19.A4 (GND), J19.A7 (DRAIN), J19.B4 (GND), J19.B7 (DRAIN), J20.11 (CKS), J20.17 (GND), J20.2 (D2S), J20.5 (D1S), J20.8 (D0S), J20.SH1 (SH), J20.SH2 (SH), J20.SH3 (SH), J20.SH4 (SH), J22.11 (CKS), J22.17 (GND), J22.2 (D2S), J22.5 (D1S), J22.8 (D0S), J22.SH1 (SH), J22.SH2 (SH), J22.SH3 (SH), J22.SH4 (SH), U1.3 (GND), U1.8 (GND), U10.3 (GND), U10.8 (GND), U11.61 (GND), U12.19 (SHIELD), U12.20 (SHIELD), U13.3 (GND)
- net QSPI_SCLK: now also U11.56 (QSPI_SCLK)
- net QSPI_SD0: now also U11.57 (QSPI_SD0)
- net QSPI_SD1: now also U11.59 (QSPI_SD1)
- net QSPI_SD2: now also U11.58 (QSPI_SD2)
- net QSPI_SD3: now also U11.55 (QSPI_SD3)
- net QSPI_SS: now also U11.60 (~{QSPI_SS})
- net RX0: now also U11.18 (GPIO14)
- net TX0: now also U11.17 (GPIO13)
- net VBUS: now also J19.A1 (VBUS), J19.B1 (VBUS)
- net XIN: now also U11.21 (XIN)
- net XOUT: now also U11.22 (XOUT)
- net USBOTG_ID: now reaches Module1.101 (USB_OTG_ID)
- net PCIE_nCLKREQ: now reaches Module1.102 (PCIe_nCLKREQ)
- net USB2_N: now reaches Module1.103 (USB2_N)
- net PCIE_nWAKE: now reaches Module1.104 (PCIE_nWAKE)
- net USB2_P: now reaches Module1.105 (USB2_P)
- net PCIE_PWR_EN: now reaches Module1.106 (PCIE_PWR_EN)
- net PCIE_nRST: now reaches Module1.109 (PCIe_nRST)
- net PCIE_CLK_P: now reaches Module1.110 (PCIe_CLK_P)
- net VBUS_EN: now reaches Module1.111 (VBUS_EN)
- net PCIE_CLK_N: now reaches Module1.112 (PCIe_CLK_N)
- net DPHY0_D0_N: now reaches Module1.115 (MIPI0_D0_N)
- net PCIE_RX_P: now reaches Module1.116 (PCIe_RX_P)
- net DPHY0_D0_P: now reaches Module1.117 (MIPI0_D0_P)
- net PCIE_RX_N: now reaches Module1.118 (PCIe_RX_N)
- net DPHY0_D1_N: now reaches Module1.121 (MIPI0_D1_N)
- net PCIE_TX_P: now reaches Module1.122 (PCIe_TX_P)
- net DPHY0_D1_P: now reaches Module1.123 (MIPI0_D1_P)
- net PCIE_TX_N: now reaches Module1.124 (PCIe_TX_N)
- net DPHY0_C_N: now reaches Module1.127 (MIPI0_C_N)
- net USB3-0-RX_N: now reaches Module1.128 (USB3-0-RX_N)
- net USB3-0-RX_N: now also J19.A6 (SSRX+)
- net DPHY0_C_P: now reaches Module1.129 (MIPI0_C_P)
- net USB3-0-RX_P: now reaches Module1.130 (USB3-0-RX_P)
- net USB3-0-RX_P: now also J19.A5 (SSRX-)
- net DPHY0_D2_N: now reaches Module1.133 (MIPI0_D2_N)
- net USB3-0-D_P: now reaches Module1.134 (USB3-0-D_P)
- net USB3-0-D_P: now also J19.A3 (D+)
- net DPHY0_D2_P: now reaches Module1.135 (MIPI0_D2_P)
- net USB3-0-D_N: now reaches Module1.136 (USB3-0-D_N)
- net USB3-0-D_N: now also J19.A2 (D-)
- net DPHY0_D3_N: now reaches Module1.139 (MIPI0_D3_N)
- net USB3-0-TX_N: now reaches Module1.140 (USB3-0-TX_N)
- net USB3-0-TX_N: now also J19.A9 (SSTX+)
- net DPHY0_D3_P: now reaches Module1.141 (MIPI0_D3_P)
- net USB3-0-TX_P: now reaches Module1.142 (USB3-0-TX_P)
- net USB3-0-TX_P: now also J19.A8 (SSTX-)
- net HDMI1_HOTPLUG: now reaches Module1.143 (HDMI1_HOTPLUG)
- net HDMI1_HOTPLUG: now also J20.19 (HPD/HEAC-)
- net HDMI1_SDA: now reaches Module1.145 (HDMI1_SDA)
- net HDMI1_SDA: now also J20.16 (SDA)
- net HDMI1_D2_P: now reaches Module1.146 (HDMI1_TX2_P)
- net HDMI1_D2_P: now also J20.1 (D2+)
- net HDMI1_SCL: now reaches Module1.147 (HDMI1_SCL)
- net HDMI1_SCL: now also J20.15 (SCL)
- net HDMI1_D2_N: now reaches Module1.148 (HDMI1_TX2_N)
- net HDMI1_D2_N: now also J20.3 (D2-)
- net HDMI1_CEC: now reaches Module1.149 (HDMI1_CEC)
- net HDMI1_CEC: now also J20.13 (CEC)
- net HDMI0_CEC: now reaches Module1.151 (HDMI0_CEC)
- net HDMI0_CEC: now also J22.13 (CEC)
- net HDMI1_D1_P: now reaches Module1.152 (HDMI1_TX1_P)
- net HDMI1_D1_P: now also J20.4 (D1+)
- net HDMI0_HOTPLUG: now reaches Module1.153 (HDMI0_HOTPLUG)
- net HDMI0_HOTPLUG: now also J22.19 (HPD/HEAC-)
- net HDMI1_D1_N: now reaches Module1.154 (HDMI1_TX1_N)
- net HDMI1_D1_N: now also J20.6 (D1-)
- net USB3-1-RX_N: now reaches Module1.157 (USB3-1-RX_N)
- net USB3-1-RX_N: now also J19.B6 (SSRX+)
- net HDMI1_D0_P: now reaches Module1.158 (HDMI1_TX0_P)
- net HDMI1_D0_P: now also J20.7 (D0+)
- net USB3-1-RX_P: now reaches Module1.159 (USB3-1-RX_P)
- net USB3-1-RX_P: now also J19.B5 (SSRX-)
- net HDMI1_D0_N: now reaches Module1.160 (HDMI1_TX0_N)
- net HDMI1_D0_N: now also J20.9 (D0-)
- net USB3-1-D_P: now reaches Module1.163 (USB3-1-D_P)
- net USB3-1-D_P: now also J19.B3 (D+)
- net HDMI1_CK_P: now reaches Module1.164 (HDMI1_CLK_P)
- net HDMI1_CK_P: now also J20.10 (CK+)
- net USB3-1-D_N: now reaches Module1.165 (USB3-1-D_N)
- net USB3-1-D_N: now also J19.B2 (D-)
- net HDMI1_CK_N: now reaches Module1.166 (HDMI1_CLK_N)
- net HDMI1_CK_N: now also J20.12 (CK-)
- net USB3-1-TX_N: now reaches Module1.169 (USB3-1-TX_N)
- net USB3-1-TX_N: now also J19.B9 (SSTX+)
- net HDMI0_D2_P: now reaches Module1.170 (HDMI0_TX2_P)
- net HDMI0_D2_P: now also J22.1 (D2+)
- net USB3-1-TX_P: now reaches Module1.171 (USB3-1-TX_P)
- net USB3-1-TX_P: now also J19.B8 (SSTX-)
- net HDMI0_D2_N: now reaches Module1.172 (HDMI0_TX2_N)
- net HDMI0_D2_N: now also J22.3 (D2-)
- net DPHY1_D0_N: now reaches Module1.175 (MIPI1_D0_N)
- net HDMI0_D1_P: now reaches Module1.176 (HDMI0_TX1_P)
- net HDMI0_D1_P: now also J22.4 (D1+)
- net DPHY1_D0_P: now reaches Module1.177 (MIPI1_D0_P)
- net HDMI0_D1_N: now reaches Module1.178 (HDMI0_TX1_N)
- net HDMI0_D1_N: now also J22.6 (D1-)
- net DPHY1_D1_N: now reaches Module1.181 (MIPI1_D1_N)
- net HDMI0_D0_P: now reaches Module1.182 (HDMI0_TX0_P)
- net HDMI0_D0_P: now also J22.7 (D0+)
- net DPHY1_D1_P: now reaches Module1.183 (MIPI1_D1_P)
- net HDMI0_D0_N: now reaches Module1.184 (HDMI0_TX0_N)
- net HDMI0_D0_N: now also J22.9 (D0-)
- net DPHY1_C_N: now reaches Module1.187 (MIPI1_C_N)
- net HDMI0_CK_P: now reaches Module1.188 (HDMI0_CLK_P)
- net HDMI0_CK_P: now also J22.10 (CK+)
- net DPHY1_C_P: now reaches Module1.189 (MIPI1_C_P)
- net HDMI0_CK_N: now reaches Module1.190 (HDMI0_CLK_N)
- net HDMI0_CK_N: now also J22.12 (CK-)
- net DPHY1_D2_N: now reaches Module1.193 (MIPI1_D2_N)
- net DPHY1_D3_N: now reaches Module1.194 (MIPI1_D3_N)
- net DPHY1_D2_P: now reaches Module1.195 (MIPI1_D2_P)
- net DPHY1_D3_P: now reaches Module1.196 (MIPI1_D3_P)
- net HDMI0_SDA: now reaches Module1.199 (HDMI0_SDA)
- net HDMI0_SDA: now also J22.16 (SDA)
- net HDMI0_SCL: now reaches Module1.200 (HDMI0_SCL)
- net HDMI0_SCL: now also J22.15 (SCL)
- net at R12.1: now also U11.52 (USB_DP)
- net at R11.1: now also U11.51 (USB_DM)
- net TRD0_N: now reaches Module1.10 (Ethernet_Pair0_N)
- net TRD0_N: now also U10.4 (D2+), U10.7, U12.2 (TRD0-)
- net CAM_GPIO1: now reaches Module1.100 (CAM_GPIO1)
- net TRD2_P: now reaches Module1.11 (Ethernet_Pair2_P)
- net TRD2_P: now also U1.5 (D2-), U1.6, U12.7 (TRD2+)
- net TRD0_P: now reaches Module1.12 (Ethernet_Pair0_P)
- net TRD0_P: now also U10.5 (D2-), U10.6, U12.1 (TRD0+)
- net ETH_LEDY: now reaches Module1.15 (Ethernet_nLED3(3.3v))
- net ETH_LEDY: now also R3.2
- net TACHO: now reaches Module1.16 (FAN_TACHO)
- net ETH_LEDG: now reaches Module1.17 (Ethernet_nLED2(3.3v))
- net ETH_LEDG: now also R2.2
- net SYNC_OUT: now reaches Module1.18 (Ethernet_SYNC_OUT(3.3v))
- net PWM: now reaches Module1.19 (FAN_PWM)
- net EEPROM_nWP: now reaches Module1.20 (EEPROM_nWP)
- net at Module1.21 (LED_nACT): now also R1.2
- net GPIO26: now reaches Module1.24 (GPIO26)
- net GPIO21: now reaches Module1.25 (GPIO21)
- net GPIO19: now reaches Module1.26 (GPIO19)
- net GPIO20: now reaches Module1.27 (GPIO20)
- net GPIO13: now reaches Module1.28 (GPIO13)
- net GPIO16: now reaches Module1.29 (GPIO16)
- net TRD3_P: now reaches Module1.3 (Ethernet_Pair3_P)
- net TRD3_P: now also U1.1 (D1+), U1.10, U12.9 (TRD3+)
- net GPIO6: now reaches Module1.30 (GPIO6)
- net GPIO12: now reaches Module1.31 (GPIO12)
- net GPIO5: now reaches Module1.34 (GPIO5)
- net ID_SC: now reaches Module1.35 (ID_SC)
- net ID_SC: now also J12.1 (Pin_1)
- net ID_SD: now reaches Module1.36 (ID_SD)
- net ID_SD: now also J12.3 (Pin_3)
- net GPIO7: now reaches Module1.37 (GPIO7)
- net GPIO11: now reaches Module1.38 (GPIO11)
- net GPIO8: now reaches Module1.39 (GPIO8)
- net TRD1_P: now reaches Module1.4 (Ethernet_Pair1_P)
- net TRD1_P: now also U10.1 (D1+), U10.10, U12.3 (TRD1+)
- net GPIO9: now reaches Module1.40 (GPIO9)
- net GPIO25: now reaches Module1.41 (GPIO25)
- net GPIO10: now reaches Module1.44 (GPIO10)
- net GPIO24: now reaches Module1.45 (GPIO24)
- net GPIO22: now reaches Module1.46 (GPIO22)
- net GPIO23: now reaches Module1.47 (GPIO23)
- net GPIO27: now reaches Module1.48 (GPIO27)
- net GPIO18: now reaches Module1.49 (GPIO18)
- net TRD3_N: now reaches Module1.5 (Ethernet_Pair3_N)
- net TRD3_N: now also U1.2 (D1-), U1.9, U12.10 (TRD3-)
- net GPIO17: now reaches Module1.50 (GPIO17)
- net GPIO15: now reaches Module1.51 (GPIO15)
- net GPIO4: now reaches Module1.54 (GPIO4)
- net GPIO14: now reaches Module1.55 (GPIO14)
- net GPIO3: now reaches Module1.56 (GPIO3)
- net SD_CLK: now reaches Module1.57 (SD_CLK)
- net GPIO2: now reaches Module1.58 (GPIO2)
- net TRD1_N: now reaches Module1.6 (Ethernet_Pair1_N)
- net TRD1_N: now also U10.2 (D1-), U10.9, U12.6 (TRD1-)
- net SD_DAT3: now reaches Module1.61 (SD_DAT3)
- net SD_CMD: now reaches Module1.62 (SD_CMD)
- net SD_DAT0: now reaches Module1.63 (SD_DAT0)
- net SD_DAT1: now reaches Module1.67 (SD_DAT1)
- net SD_DAT2: now reaches Module1.69 (SD_DAT2)
- net SD_PWR_ON: now reaches Module1.75 (SD_PWR_ON)
- net VBAT: now reaches Module1.76 (VBAT)
- net +5v: now reaches Module1.77 (+5v_(Input))
- net +5v: now also Module1.79 (+5v_(Input)), Module1.81 (+5v_(Input)), Module1.83 (+5v_(Input)), Module1.85 (+5v_(Input)), Module1.87 (+5v_(Input)), C12.1, U13.1 (IN)
- net GPIO_VREF: now reaches Module1.78 (GPIO_VREF(1.8v/3.3v_Input))
- net GPIO_VREF: now also R6.1, R7.1
- net SCL0: now reaches Module1.80 (SCL0)
- net SDA0: now reaches Module1.82 (SDA0)
- net +3.3v: now reaches Module1.84 (+3.3v_(Output))
- net +3.3v: now also Module1.86 (+3.3v_(Output)), D2.2 (A), U12.15 (LEDY_A), U12.17 (LEDG_A)
- net +1.8v: now reaches Module1.88 (+1.8v_(Output))
- net +1.8v: now also Module1.90 (+1.8v_(Output))
- net WL_nDis: now reaches Module1.89 (WiFi_nDisable)
- net WL_nDis: now also J17.1 (Pin_1)
- net TRD2_N: now reaches Module1.9 (Ethernet_Pair2_N)
- net TRD2_N: now also U1.4 (D2+), U1.7, U12.8 (TRD2-)
- net BT_nDis: now reaches Module1.91 (BT_nDisable)
- net BT_nDis: now also J17.3 (Pin_3)
- net PWR_BUT: now reaches Module1.92 (PWR_BUT)
- net nRPIBOOT: now reaches Module1.93 (nRPIBOOT)
- net CC1: now reaches Module1.94 (CC1)
- net nPWR_LED: now reaches Module1.95 (LED_nPWR)
- net CC2: now reaches Module1.96 (CC2)
- net CAM_GPIO0: now reaches Module1.97 (CAM_GPIO0)
- net PMIC_ENABLE: now reaches Module1.99 (PMIC_ENABLE)
- new net: R2.1, U12.16 (LEDY_K)
- new net: D2.1 (K), R1.1, TP3.1
- new net: R3.1, U12.18 (LEDG_K)
- new net: J11.A1 (GND), J11.A12 (GND), J11.B1 (GND), J11.B12 (GND)
- new net: J11.A4 (VBUS), J11.A9 (VBUS), J11.B4 (VBUS), J11.B9 (VBUS)
- new net: U11.23 (DVDD), U11.39 (DVDD), U11.6 (DVDD)
- new net: C3.1, U12.4 (CT), U12.5 (CT)
- new net HDMI_5v: C13.1, J20.18 (+5V), J22.18 (+5V), U13.2 (OUT)
- new net SCL1: J12.2 (Pin_2), R7.2
- new net SDA1: J12.4 (Pin_4), R6.2
- new net TR0_TAP: J18.3 (Pin_3), U12.11 (VC1)
- new net TR1_TAP: J18.1 (Pin_1), U12.12 (VC2)
- new net TR2_TAP: J18.2 (Pin_2), U12.13 (VC3)
- new net TR3_TAP: J18.4 (Pin_4), U12.14 (VC4)
- no-connect marks 0 -> 3
Other:
- note added: "Activity LED"
- note added: "Ethernet"
- note added: "Ethernet POE Protection"
- note added: "Jumpers to be fitted if DPHY1 is used"
- note added: "Not Fitted header"
- note added: "POE Header"
- note added: "Stacked USB connectors"
- note added: "USB 3 Pairs P/N swapped to help routing"
- moved on the sheet: Module1B
