File: PCB/stick2/stick2/stick2.kicad_sch (KiCad schematic)
At the start: 13 parts, among them J1 Conn_01x08_Pin, U1 MLX90395xLW

Commit message: boards
Parts:
- removed J1: Conn_01x08_Pin, Connector_PinHeader_2.54mm:PinHeader_1x08_P2.54mm_Horizontal, symbol Connector:Conn_01x08_Pin
- removed R4: 100, Resistor_SMD:R_0603_1608Metric_Pad0.98x0.95mm_HandSolder, symbol Device:R_US
- added C10, C14, C15, C16, C20, C21, C23, C24, C25, C26, C27: 100n, RPI_COMPILED:generic_capc1005x50, symbol RPI_DB:Capacitors | MLCC | M1005/RP-01BJ9Y-KRGF41
- added C11, C22, C9: 10u, RPI_COMPILED:generic_capc2012x125, symbol RPI_DB:Capacitors | MLCC | M2012/RP-01GYSK-AVBE41
- added C12, C13: 15p, RPI_COMPILED:generic_capc1005x50, symbol RPI_DB:Capacitors | MLCC | M1005/RP-01C89W-LLY9XV
- added C17, C18: 4.7u, RPI_COMPILED:generic_capc1005x50_wide, symbol RPI_DB:Capacitors | MLCC | M1005/RP-019A1P-0C2GHY
- added C19: 4.7u, RPI_COMPILED:generic_capc1005x50, symbol RPI_DB:Capacitors | MLCC | M1005/RP-019A1P-0C2GHY
- added H3, H4, H5, H6: MountingHole, MountingHole:MountingHole_2.2mm_M2, symbol Mechanical:MountingHole
- added J1: Conn_01x04_Pin, Connector_PinHeader_2.54mm:PinHeader_1x04_P2.54mm_Horizontal, symbol Connector:Conn_01x04_Pin
- added J2: Conn_01x16, Connector_PinHeader_2.54mm:PinHeader_1x16_P2.54mm_Horizontal, symbol Connector_Generic:Conn_01x16
- added J3: USB_C_Receptacle_USB2.0_16P, Connector_USB:USB_C_Receptacle_GCT_USB4110, symbol Connector:USB_C_Receptacle_USB2.0_16P
- added J4: Conn_01x06_Pin, Connector_PinHeader_2.54mm:PinHeader_1x06_P2.54mm_Horizontal, symbol Connector:Conn_01x06_Pin
- added J5: Conn_01x03_Pin, Connector_PinHeader_2.54mm:PinHeader_1x03_P2.54mm_Horizontal, symbol Connector:Conn_01x03_Pin
- added L1: 3.3u, RPI_COMPILED:abracon_aota-b201610s3r3-101-t, symbol RPI_DB:Inductors | Fixed | M2016/RP-01GY5D-2VC7WP
- added R1: 10k, RPI_COMPILED:generic_resc1005x35, symbol RPI_DB:Resistors | Chip | M1005/RP-019A1P-53DHSX
- added R10, R9: 0, RPI_COMPILED:generic_resc1005x35, symbol RPI_DB:Resistors | Chip | M1005/RP-019A1P-4Y4V63
- added R11, R12: 5.1k, Resistor_SMD:R_0603_1608Metric_Pad0.98x0.95mm_HandSolder, symbol Device:R_US
- added R2, R5, R6: 1k, RPI_COMPILED:generic_resc1005x35, symbol RPI_DB:Resistors | Chip | M1005/RP-019A1P-4Z6ZWY
- added R3: 33, RPI_COMPILED:generic_resc1005x35, symbol RPI_DB:Resistors | Chip | M1005/RP-019A1P-58PW9L
- added R7, R8: 27, RPI_COMPILED:generic_resc1005x35, symbol RPI_DB:Resistors | Chip | M1005/RP-01C89V-LTEYC4
- added SW1, SW2: 434133025816, RPI_COMPILED:wurthelek_434133025816, symbol RPI_DB:Electromechanical | Switches | Tactile/RP-01H0MT-6E9H8F
- added U2: NCP1117ST33T3G, RPI_COMPILED:onsemi_ncp1117st33t3g, symbol RPI_DB:Integrated_Circuits | Power | LDO/RP-01JWD9-7JRX6J
- added U3: W25Q128JVSIQ, RPI_COMPILED:generic_soic127p790x195-8, symbol RPI_DB:Integrated_Circuits | Memory | Serial_Flash | SPI/RP-01JWD4-F1H4N9
- added U4: RP2350A, RPI_COMPILED:rpi_rp2350a_vias, symbol RPI_DB:Integrated_Circuits | Microcontrollers/RP-01HA9H-9K5E8T
- added X1: 12MHz, RPI_COMPILED:generic_xtalcc320x250x80-4, symbol RPI_DB:Frequency_Timing | Crystals/RP-01G8X7-GS352B
- C1, C2, C3, C4, C5, C6, C7, C8: KiLib_Generator (none) -> SMD_2terminal_chip_molded
- H1, H2: KiLib_Generator (none) -> mounting_hardware/mounting_hole
- U1: KiLib_Generator (none) -> package/no_lead
Connections:
- net GPIO27_ADC1: now reaches C2.1, U1.3 (SCLK)
- net GPIO27_ADC1: now also U4.41 (GPIO27_ADC1)
- net CS: no longer names the net of C8.1, U1.2 (~{CS})
- net MISO: no longer names the net of C4.1, U1.6 (MISO)
- net MOSI renamed GPIO26_ADC0
- net GPIO26_ADC0: now also U4.40 (GPIO26_ADC0)
- new net: C13.1, R2.2, X1.3
- new net: R5.1, SW2.1, SW2.2
- new net: R7.2, U4.52 (USB_DP)
- new net: J3.A5 (CC1), R11.1
- new net: J3.B5 (CC2), R12.1
- new net: R8.2, U4.51 (USB_DM)
- new net +1V1: C14.1, C15.1, C16.1, C17.1, L1.1, U4.23 (DVDD), U4.39 (DVDD), U4.50 (VREG_FB), U4.6 (DVDD)
- new net +3V3: C10.1, C11.1, C18.1, C20.1, C21.1, C22.1, C23.1, C24.1, C25.1, C26.1, C27.1, J2.4 (Pin_4), R1.1, R3.1, U2.2 (OUT), U2.4 (OUT), U3.8 (VCC), U4.1 (IOVDD), U4.11 (IOVDD), U4.20 (IOVDD), U4.30 (IOVDD), U4.38 (IOVDD), U4.44 (ADC_AVDD), U4.45 (IOVDD), U4.49 (VREG_VIN), U4.53 (USB_OTP_VDD), U4.54 (QSPI_IOVDD)
- new net COM: J2.9 (Pin_9), U4.32 (GPIO20)
- new net DATA: J5.2 (Pin_2), U4.15 (GPIO11)
- new net Down: J2.16 (Pin_16), U4.18 (GPIO14)
- new net FLASH_SS: R1.2, R10.2, R9.2, U3.1 (~{CS})
- new net GND: C10.2, C11.2, C12.2, C13.2, C14.2, C15.2, C16.2, C17.2, C18.2, C19.2, C20.2, C21.2, C22.2, C23.2, C24.2, C25.2, C26.2, C27.2, C9.2, J1.1 (Pin_1), J2.1 (Pin_1), J3.A1 (GND), J3.A12 (GND), J3.B1 (GND), J3.B12 (GND), J3.S1 (SHIELD), J5.3 (Pin_3), R11.2, R12.2, R5.2, SW1.1, SW1.2, U2.1 (GND), U3.4 (GND), U4.47 (VREG_PGND), U4.61 (GND), X1.2, X1.4
- new net GPIO0: R9.1, U4.2 (GPIO0)
- new net GPIO1: U4.3 (GPIO1)
- new net GPIO10: U4.14 (GPIO10)
- new net GPIO12: J2.13 (Pin_13), U4.16 (GPIO12)
- new net GPIO13: J2.14 (Pin_14), U4.17 (GPIO13)
- new net GPIO15: J2.15 (Pin_15), U4.19 (GPIO15)
- new net GPIO16: U4.27 (GPIO16)
- new net GPIO17: J2.10 (Pin_10), U4.28 (GPIO17)
- new net GPIO18: J2.11 (Pin_11), U4.29 (GPIO18)
- new net GPIO19: J2.12 (Pin_12), U4.31 (GPIO19)
- new net GPIO2: U4.4 (GPIO2)
- new net GPIO21: J2.8 (Pin_8), U4.33 (GPIO21)
- new net GPIO22: J2.7 (Pin_7), U4.34 (GPIO22)
- new net GPIO23: J2.6 (Pin_6), U4.35 (GPIO23)
- new net GPIO24: J2.5 (Pin_5), U4.36 (GPIO24)
- new net GPIO25: U4.37 (GPIO25)
- new net GPIO28_ADC2: U4.42 (GPIO28_ADC2)
- new net GPIO29_ADC3: U4.43 (GPIO29_ADC3)
- new net GPIO3: U4.5 (GPIO3)
- new net GPIO4: U4.7 (GPIO4)
- new net GPIO5: U4.8 (GPIO5)
- new net GPIO6: U4.9 (GPIO6)
- new net GPIO7: U4.10 (GPIO7)
- new net GPIO8: U4.12 (GPIO8)
- new net GPIO9: U4.13 (GPIO9)
- new net QSPI_SCLK: U3.6 (CLK), U4.56 (QSPI_SCLK)
- new net QSPI_SD0: U3.5 (DI_IO0), U4.57 (QSPI_SD0)
- new net QSPI_SD1: U3.2 (DO_IO1), U4.59 (QSPI_SD1)
- new net QSPI_SD2: U3.3 (~{WP}_IO2), U4.58 (QSPI_SD2)
- new net QSPI_SD3: U3.7 (~{HOLD}_IO3), U4.55 (QSPI_SD3)
- new net QSPI_SS: R10.1, R6.1, U4.60 (QSPI_~{SS})
- new net RUN: SW2.3, SW2.4, U4.26 (RUN)
- new net SWCLK: U4.24 (SWCLK)
- new net SWD: U4.25 (SWDIO)
- new net USB_D+: J1.2 (Pin_2), J3.A6 (D+), J3.B6 (D+), R7.1
- new net USB_D-: J1.3 (Pin_3), J3.A7 (D-), J3.B7 (D-), R8.1
- new net VBUS: C9.1, J1.4 (Pin_4), J2.2 (Pin_2), J2.3 (Pin_3), J3.A4 (VBUS), J3.A9 (VBUS), J3.B4 (VBUS), J3.B9 (VBUS), J5.1 (Pin_1), U2.3 (IN)
- new net VREG_AVDD: C19.1, R3.2, U4.46 (VREG_AVDD)
- new net VREG_LX: L1.2, U4.48 (VREG_LX)
- new net XIN: C12.1, U4.21 (XIN), X1.1
- new net XOUT: R2.1, U4.22 (XOUT)
- new net ~{USB_BOOT}: R6.2, SW1.3, SW1.4
Other:
- note added: "12MHz Crystal"
- note added: "BOOTSEL Button"
- note added: "Flash"
- note added: "If using RP2354 (internal flash), remove R10. R9 can be fit to use U3 as secondary memory."
- note added: "Make sure R7 and R8 are close to RP2350"
- note added: "Power"
- note added: "RUN Button"
- moved on the sheet: H1, H2
