File: PCB/stick2/stick2-IO/stick2-IO.kicad_pcb (KiCad board)
At the start: 2 copper layers, 76 x 42.1 mm, 20 parts, among them J10 Conn_01x12_Pin, J11 Conn_01x04_Pin, J12 Conn_01x05_Pin, J13 Conn_01x16_Pin, J2 Conn_02x04_Row_Letter_Last, J3 Conn_02x04_Row_Letter_Last, J4 Conn_02x04_Row_Letter_Last, J5 Conn_02x04_Row_Letter_Last, J6 Conn_02x04_Row_Letter_Last, J7 Conn_02x04_Row_Letter_Last, J8 Conn_02x04_Row_Letter_Last, J9 Conn_02x04_Row_Letter_Last, U2 TLC5947RHB, U3 TLC5947RHB, U6 CD74HC4067M

Commit message: stopping point
Parts:
- moved H4 2.00 mm to (173.0, 87.5)
- moved H6 2.00 mm to (102.0, 87.5)
- moved U6 1.12 mm to (140.0, 85.0)
- moved J12 1.00 mm to (110.1, 87.0)
Routing:
- net Net-(J10-Pin_6): track 27.2 -> 62.9 mm
- net Net-(J10-Pin_9): track 38.7 -> 74.2 mm
- net Net-(J10-Pin_7): track 30.1 -> 61.4 mm
- net Net-(J10-Pin_8): track 32.9 -> 59.8 mm
- net Net-(J10-Pin_10): track 44.4 -> 61.9 mm
- net Net-(J10-Pin_11): track 49.8 -> 61.1 mm
- net /S2: track 88.6 -> 92.8 mm
- net /GND: track 11.7 -> 8.21 mm, vias 10 -> 18
- net /S3: track 90.0 -> 93.4 mm
- net /S1: track 84.7 -> 87.7 mm
- net /S0: track 83.2 -> 85.9 mm
- net /SCLK: track 52.9 -> 50.6 mm
- net /Right: track 69.8 -> 67.6 mm
- net /XLAT: track 48.9 -> 46.7 mm
- net Net-(J11-Pin_1): track 33.6 -> 31.5 mm
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- added copper zone on F.Cu, net /GND
Other:
- board size 76 x 42.1 mm -> 76 x 40.1 mm
