File: PCB/stick2/stick2-IO/stick2-IO.kicad_sch (KiCad schematic)
At the start: 20 parts, among them J10 Conn_01x12_Pin, J11 Conn_01x04_Pin, J12 Conn_01x05_Pin, J13 Conn_01x16_Pin, J2 Conn_02x04_Row_Letter_Last, J3 Conn_02x04_Row_Letter_Last, J4 Conn_02x04_Row_Letter_Last, J5 Conn_02x04_Row_Letter_Last, J6 Conn_02x04_Row_Letter_Last, J7 Conn_02x04_Row_Letter_Last, J8 Conn_02x04_Row_Letter_Last, J9 Conn_02x04_Row_Letter_Last, U2 TLC5947RHB, U3 TLC5947RHB, U6 CD74HC4067M

Commit message: stopping point
Parts:
- H3, H4, H5, H6: KiLib_Generator (none) -> mounting_hardware/mounting_hole
- J13: footprint Connector_PinHeader_2.54mm:PinHeader_1x16_P2.54mm_Vertical -> Connector_PinSocket_2.54mm:PinSocket_1x16_P2.54mm_Vertical
Changed lines of the file:
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@@
+			)
+		)
+		(property "KiLib_Generator" "mounting_hardware/mounting_hole"
+			(at 81.28 -20.32 0)
+			(hide yes)
+			(show_name no)
+			(do_not_autoplace no)
+			(effects
+				(font
+					(size 1.27 1.27)
+				)
 			)
 		)
@@
 			)
 		)
+		(property "KiLib_Generator" "mounting_hardware/mounting_hole"
+			(at 80.01 -27.94 0)
+			(hide yes)
+			(show_name no)
+			(do_not_autoplace no)
+			(effects
+				(font
+					(size 1.27 1.27)
+				)
+			)
+		)
 		(instances
 			(project "stick2-IO"
@@
 			)
 		)
+		(property "KiLib_Generator" "mounting_hardware/mounting_hole"
+			(at 82.55 -11.43 0)
+			(hide yes)
+			(show_name no)
+			(do_not_autoplace no)
+			(effects
+				(font
+					(size 1.27 1.27)
+				)
+			)
+		)
 		(instances
 			(project "stick2-IO"
@@
 			)
 		)
+		(property "KiLib_Generator" "mounting_hardware/mounting_hole"
+			(at 80.01 -34.29 0)
+			(hide yes)
+			(show_name no)
+			(do_not_autoplace no)
+			(effects
+				(font
+					(size 1.27 1.27)
+				)
+			)
+		)
 		(instances
 			(project "stick2-IO"
@@
 			)
 		)
-		(property "Footprint" "Connector_PinHeader_2.54mm:PinHeader_1x16_P2.54mm_Vertical"
+		(property "Footprint" "Connector_PinSocket_2.54mm:PinSocket_1x16_P2.54mm_Vertical"
 			(at 26.67 111.76 0)
 			(hide yes)
@@
 			)
 		)
-		(property "Description" "Generic connector, single row, 01x16, script generated"
+		(property "Description" ""
 			(at 26.67 111.76 0)
 			(hide yes)
